File: PCB/PCB.kicad_pcb (KiCad board)
At the start: 4 copper layers, 76.5 x 65 mm, 31 parts, among them J1 ESP_Left, J2 ESP_Right, J3 Term Block, J4 Term Block, J5 Term Block, U1 ISO6740, U2 ISO6740

Commit message: first test with case
Parts:
- JP1, JP2: footprint Jumper:SolderJumper-2_P1.3mm_Open_TrianglePad1.0x1.5mm -> Jumper:SolderJumper-2_P1.3mm_Open_RoundedPad1.0x1.5mm
Other:
- board text added: "01"
- board text added: "02"
- board text added: "04"
- board text added: "06"
- board text added: "12V"
- board text added: "34"
- board text added: "36"
- board text added: "38"
- board text added: "40"
- board text added: "5V"
- board text added: "GND1"
- board text added: "GND2"
